Commit message: Draw the R1 forearm without the stock fist the Dex3 replaces
The upstream wrist_roll_link mesh is the forearm tube (x < 0.080 m) plus the stock fist
(0.080-0.143 m), which rendered through the Dex3 palm mounted at 0.080 m. The build now
cuts the mesh at the Dex3 mount (*_wrist_roll_link_forearm.STL) and uses it as the wrist
visual in the URDF and MJCF, as BruteForce's r1_dex3_constants.py removes the fist.
Collision (forearm cylinder + Dex3 hulls) and mass are unchanged. The hands stay fixed,
as on NVIDIA's released G1 (g1_model_12_dex). Test: the wrist visual ends at the mount.

File: gear_sonic/data/assets/robot_description/urdf/r1/r1_dex3.urdf (robot description, URDF)
Before this commit: robot r1_dex3, 56 links, 55 joints
Links:
- link left_wrist_roll_link: geometry collision cylinder length=0.08 radius=0.03; visual mesh filename=meshes/left_wrist_roll_link_forearm.STL
- link right_wrist_roll_link: geometry collision cylinder length=0.08 radius=0.03; visual mesh filename=meshes/right_wrist_roll_link_forearm.STL

Commit message: Calm teleop: no-balance-step rewards (stage B3), semi-closed Dex3 hands, calmer runtime
Rewards (mdp/smoothness.py, preset sonic_r1_dex3_teleop_calm.yaml):
- stance_foot_motion: |v_foot - v_foot_ref|^2 while the reference foot stands,
  against balance steps, shuffles and sliding;
- leg_joint_vel_error: sum (dq - dq_ref)^2 over the legs.
Both are zero under perfect tracking.

Smooth preset corrected after stage B2 lost tracking (uniform success
0.845 -> 0.706 in 1000 iterations, walking clips 0.75 -> 0.47):
- L2C2 had interpolated the tokenizer, making the FSQ encoder resist reference
  changes; it now interpolates the proprioception only (l2c2_keys), at 0.5;
- leg action-rate multipliers are down to 1.5-2.

Hands: r1_spec.DEX3_HOLD_POSE, a relaxed semi-closed fist, is baked into
the fixed finger joints of the URDF/MJCF. On the real robot the DDS process
publishes rt/dex3/{left,right}/cmd (hands.py): the hold pose by default;
grip points, grip + trigger makes a fist, trigger pinches, A/X opens.

Runtime (run.py defaults):
- walking <= 0.5 m/s and turning <= 0.6 rad/s;
- a critically damped, speed-limited joint-space filter on the IK targets;
- the planner holds the stand-up stance until the sticks first move (its
  first idle plan shuffled the feet 10 cm);
- --input keys drives walking and gestures from the keyboard.

MuJoCo: elliptic friction cones with impratio 10. The default soft friction
let standing feet creep 56 mm in 20 s.
sim_gate reports unplanned_steps and idle_foot_drift_mm.

File: gear_sonic/data/assets/robot_description/urdf/r1/r1_dex3.urdf (robot description, URDF)
Before this commit: robot r1_dex3, 56 links, 55 joints
Joints:
- joint left_hand_index_0_joint: origin xyz=0.0777 0.0016 0.0285 rpy=0 0 0 -> xyz=0.0777 0.0016 0.0285 rpy=0 0 -0.8
- joint left_hand_index_1_joint: origin xyz=0.0458 0 0 rpy=0 0 0 -> xyz=0.0458 0 0 rpy=0 0 -0.9
- joint left_hand_middle_0_joint: origin xyz=0.0777 0.0016 -0.0285 rpy=0 0 0 -> xyz=0.0777 0.0016 -0.0285 rpy=0 0 -0.8
- joint left_hand_middle_1_joint: origin xyz=0.0458 0 0 rpy=0 0 0 -> xyz=0.0458 0 0 rpy=0 0 -0.9
- joint left_hand_thumb_1_joint: origin xyz=-0.0025 -0.0193 0 rpy=0 0 0 -> xyz=-0.0025 -0.0193 0 rpy=0 0 0.3
- joint left_hand_thumb_2_joint: origin xyz=0 -0.0458 0 rpy=0 0 0 -> xyz=0 -0.0458 0 rpy=0 0 0.7
- joint right_hand_index_0_joint: origin xyz=0.0777 -0.0016 0.0285 rpy=0 0 0 -> xyz=0.0777 -0.0016 0.0285 rpy=0 0 0.8
- joint right_hand_index_1_joint: origin xyz=0.0458 0 0 rpy=0 0 0 -> xyz=0.0458 0 0 rpy=0 0 0.9
- joint right_hand_middle_0_joint: origin xyz=0.0777 -0.0016 -0.0285 rpy=0 0 0 -> xyz=0.0777 -0.0016 -0.0285 rpy=0 0 0.8
- joint right_hand_middle_1_joint: origin xyz=0.0458 0 0 rpy=0 0 0 -> xyz=0.0458 0 0 rpy=0 0 0.9
- joint right_hand_thumb_1_joint: origin xyz=-0.0025 0.0193 0 rpy=0 0 0 -> xyz=-0.0025 0.0193 0 rpy=0 0 -0.3
- joint right_hand_thumb_2_joint: origin xyz=0 0.0458 0 rpy=0 0 0 -> xyz=0 0.0458 0 rpy=0 0 -0.7
